Commit message: urdf support for multi robots

File: description/alpha/urdf/alpha_5.urdf.xacro (robot description, xacro)
@@ -7,5 +7,5 @@
             <child link="${name}_base_link" />
         </joint>
-        <material name="alpha_black">
+        <material name="${name}_black">
             <color rgba="0.3 0.3 0.3 1"/>
         </material>
@@ -22,5 +22,5 @@
                 </geometry>
                 <origin rpy="0 0 0" xyz="0 0 0"/>
-                <material name="alpha_black"/>
+                <material name="${name}_black"/>
             </visual>
             <collision>
@@ -61,5 +61,5 @@
             <origin xyz="0 0 0.014"/>
             <axis xyz="0 0 1"/>
-            <limit effort="9.0" lower="0.0" upper="6.3" velocity="0.5"/>
+            <limit effort="9.0" lower="0.0" upper="5.7" velocity="0.5"/>
         </joint>
         <link name="${name}_m2_joint_link">
@@ -100,5 +100,5 @@
             <origin xyz="-0.02 0 0.033"/>
             <axis xyz="0 1 0"/>
-            <limit effort="9.0" lower="0.0" upper="3.8" velocity="0.5"/>
+            <limit effort="9.0" lower="1.5" upper="3.4" velocity="0.5"/>
         </joint>
         <link name="${name}_m2_1_2_link">
@@ -127,5 +127,5 @@
             <origin xyz="-0.04 0 -0.1453" rpy="0 0 3.14159"/>
             <axis xyz="0 1 0"/>
-            <limit effort="9.0" lower="0.0" upper="3.5" velocity="0.5"/>
+            <limit effort="9.0" lower="0.2" upper="3.4" velocity="0.5"/>
         </joint>
         <link name="${name}_m1_link">
@@ -154,5 +154,5 @@
             <origin xyz="0.02 0 0.033" rpy="0 0 2.09439"/>
             <axis xyz="0 0 -1"/>
-            <limit effort="9.0" lower="0.0" upper="6.2" velocity="0.5"/>
+            <limit effort="9.0" lower="0.0" upper="5.7" velocity="0.5"/>
         </joint>
         <material name="${name}_jaws_black">

File: description/ros2_control/vehicle_system_multi_interface.ros2_control.xacro (robot description, xacro)
@@ -60,5 +60,5 @@
         <state_interface name="current"/>
       </joint>
-      <gpio name="${prefix}_IOs">
+      <gpio name="${prefix}IOs">
         <command_interface name="position.x"/>
         <command_interface name="position.y"/>

File: description/xacro/robot_system_multi_interface.urdf.xacro (robot description, xacro)
@@ -3,29 +3,63 @@
   <!-- Enable setting arguments from the launch file -->
   <xacro:arg name="use_mock_hardware" default="true"/>
-  <xacro:arg name="prefix" default="alpha" />
+  <xacro:arg name="robot_count" default="1"/>
   <xacro:arg name="serial_port" default="/dev/ttyUSB0"/>
   <xacro:arg name="state_update_frequency" default="250"/>
-    <!-- Properties -->
-  <xacro:property name="description_package" value="ros2_control_blue_reach_5" />
-  <xacro:property name="prefix" value="$(arg prefix)" />
+  <xacro:arg name="description_package" default="ros2_control_blue_reach_5"/>
+  <!-- Properties -->
+  <xacro:property name="description_package" value="$(arg description_package)"/>
+  <xacro:property name="robot_count" value="$(arg robot_count)"/>
+  <xacro:property name="serial_port" value="$(arg serial_port)"/>
+  <xacro:property name="state_update_frequency" value="$(arg state_update_frequency)"/>
+  <xacro:property name="use_mock_hardware" value="$(arg use_mock_hardware)"/>
+  <!-- Define constants -->
+  <xacro:property name="d_min" value="1.0"/>
   <!-- Imports -->
- <xacro:include filename="$(find ${description_package})/xacro/urdf.xacro"/>
+  <xacro:include filename="$(find ros2_control_blue_reach_5)/xacro/world.xacro"/>
+  <xacro:include filename="$(find ${description_package})/xacro/urdf.xacro"/>
   <!-- Import RRBot ros2_control description -->
   <xacro:include filename="$(find ${description_package})/ros2_control/robot_system_multi_interface.ros2_control.xacro" />
   <!-- Import RRBot ros2_control description -->
   <xacro:include filename="$(find ${description_package})/ros2_control/vehicle_system_multi_interface.ros2_control.xacro" />
-  <xacro:bluerov2_heavy_alpha_urdf
-    prefix="${prefix}"/>
-  <xacro:robot_system_multi_interface
-    name="ReachSystemMultiInterface"
-    prefix="$(arg prefix)"
-    serial_port="$(arg serial_port)"
-    state_update_frequency="$(arg state_update_frequency)"
-    use_mock_hardware="$(arg use_mock_hardware)"/>
-  <xacro:vehicle_system_multi_interface
-    name="BlueSystemMultiInterface"
-    prefix="$(arg prefix)"
-    serial_port="$(arg serial_port)"
-    state_update_frequency="$(arg state_update_frequency)"
-    use_mock_hardware="$(arg use_mock_hardware)"/>
+  <!-- Instantiate the world -->
+  <xacro:sim_world/>
+  <!-- Recursive Macro Definition -->
+  <xacro:macro name="instantiate_robots" params="index count">
+    <xacro:if value="${index &lt; count}">
+      <!-- Generate prefix for the current robot -->
+      <xacro:property name="prefix" value="robot_${index + 1}_"/>
+      <!-- Compute positions and orientations -->
+      <xacro:property name="angle" value="${2 * pi * index / count}"/>
+      <!-- Compute circumference and radius -->
+      <xacro:property name="circumference" value="${count * d_min}"/>
+      <xacro:property name="radius" value="${circumference / (2 * pi)}"/>
+      <xacro:property name="x_pos" value="${radius * cos(angle)}"/>
+      <xacro:property name="y_pos" value="${radius * sin(angle)}"/>
+      <!-- Instantiate the robot -->
+      <xacro:bluerov2_heavy_alpha_urdf
+        prefix="${prefix}"
+        x="${x_pos}"
+        y="${y_pos}"
+        z="0.0"
+        rot_r="0.0"
+        rot_p="0.0"
+        rot_y="${angle}"/>
+    <xacro:robot_system_multi_interface
+      name="ReachSystemMultiInterface"
+      prefix="${prefix}"
+      serial_port="${serial_port}"
+      state_update_frequency="${state_update_frequency}"
+      use_mock_hardware="${use_mock_hardware}"/>
+    <xacro:vehicle_system_multi_interface
+      name="BlueSystemMultiInterface"
+      prefix="${prefix}"
+      serial_port="${serial_port}"
+      state_update_frequency="${state_update_frequency}"
+      use_mock_hardware="${use_mock_hardware}"/>
+      <!-- Recursively call the macro for the next robot -->
+      <xacro:instantiate_robots index="${index + 1}" count="${count}"/>
+    </xacro:if>
+  </xacro:macro>
+  <!-- Start the robot instantiation recursion -->
+  <xacro:instantiate_robots index="0" count="${int(robot_count)}"/>
 </robot>

File: description/xacro/urdf.xacro (robot description, xacro)
@@ -1,71 +1,5 @@
 <?xml version="1.0"?>
 <robot xmlns:xacro="http://ros.org/wiki/xacro">
-  <xacro:macro name="bluerov2_heavy_alpha_urdf" params="prefix">
-    <!-- world origin -->
-    <link name="world">
-        <visual>
-        <origin rpy="0 0 0" xyz="0 0 0"/>
-        <geometry>
-            <cylinder radius="0.06" length="0.09"/>
-        </geometry>
-        </visual>
-    </link>
-    <link name="world_bottom"/>
-    <link name="bathymetry_shipwreck">
-      <visual>
-        <origin xyz="0 0 0" rpy="${pi/2} 0 0"/>
-        <geometry>
-          <mesh filename="file://$(find ros2_control_blue_reach_5)/Bathymetry/meshes/manhomansett.stl" scale="5 5 5"/>
-        </geometry>
-        <material name="gray">
-          <color rgba="0.5 0.5 0.5 1.0"/>
-        </material>
-      </visual>
-      <collision>
-        <origin xyz="0 0 0" rpy="${pi/2} 0 0"/>
-        <geometry>
-          <mesh filename="file://$(find ros2_control_blue_reach_5)/Bathymetry/meshes/manhomansett.stl" scale="5 5 5"/>
-        </geometry>
-      </collision>
-    </link>
-    <!-- <link name="bathymetry_seafloor">
-      <visual>
-        <origin xyz="0 0 0" rpy="0 0 0"/>
-        <geometry>
-          <mesh filename="file://$(find ros2_control_blue_reach_5)/Bathymetry/meshes/hawaii.stl" scale="0.4 0.4 0.4"/>
-        </geometry>
-        <material name="gray">
-          <color rgba="0.5 0.5 0.5 1.0"/>
-        </material>
-      </visual>
-      <collision>
-        <origin xyz="0 0 0" rpy="0 0 0"/>
-        <geometry>
-          <mesh filename="file://$(find ros2_control_blue_reach_5)/Bathymetry/meshes/hawaii.stl" scale="0.4 0.4 0.4"/>
-        </geometry>
-      </collision>
-    </link> -->
-    <joint name="world_bottom_joint" type="fixed">
-      <child link="world_bottom" />
-      <parent link="world" />
-      <origin xyz="0.0 0.0 -8.0" rpy="0 0 0"/>
-    </joint>
-    <!-- <joint name="bathymetry_seafloor_joint" type="fixed">
-      <child link="bathymetry_seafloor"/>
-      <parent link="world_bottom" />
-      <origin xyz="0.0 0.0 0.0" rpy="0 0 0"/>
-    </joint> -->
-   <joint name="bathymetry_shipwreck_joint" type="fixed">
-      <child link="bathymetry_shipwreck" />
-      <parent link="world_bottom" />
-      <origin xyz="-15.0 -6.0 -1.0" rpy="0 0 0"/>
-    </joint>
-    <!-- Robot body origin -->
-    <link name="base_link"/>
-    <joint name="world_joint" type="fixed">
-      <child link="base_link" />
-      <parent link="world" />
-      <origin xyz="0.0 0.0 0.0" rpy="0 0 0"/>
-    </joint>
+  <xacro:macro name="bluerov2_heavy_alpha_urdf" params="prefix x:=0.0 y:=0.0 z:=2.0 rot_r:=0.0 rot_p:=0.0 rot_y:=0.0">
     <link name="${prefix}manipulator_mount_link">
       <visual>
@@ -126,5 +60,5 @@
       <child link="${prefix}base_link" />
       <parent link="base_link" />
-      <origin xyz="0.0 0.0 0.0" rpy="0 0 0"/>
+      <origin xyz="${x} ${y} ${z}" rpy="${rot_r} ${rot_p} ${rot_y}"/>
     </joint>
     <joint name="${prefix}manipulator_mount_joint" type="fixed">
@@ -142,9 +76,9 @@
     <xacro:include filename="$(find ros2_control_blue_reach_5)/blue/xacro/bluerov2_heavy_reach/urdf.xacro" />
     <!-- Instantiate the Alpha -->
-    <xacro:alpha_5 parent="${prefix}manipulator_mount_link" name="$(arg prefix)">
+    <xacro:alpha_5 parent="${prefix}manipulator_mount_link" name="${prefix}">
     <origin xyz="0 0 0" rpy="${pi} 0 0" />
     </xacro:alpha_5>
     <!-- Instantiate the BlueROV2 -->
-    <xacro:bluerov2_heavy_reach_urdf prefix="$(arg prefix)" />
+    <xacro:bluerov2_heavy_reach_urdf prefix="${prefix}"/>
   </xacro:macro>
 </robot>
