Commit message: dynamic controller yaml generation

File: description/xacro/world.xacro (robot description, xacro)
@@ -59,5 +59,5 @@
       <child link="bathymetry_shipwreck" />
       <parent link="world_bottom" />
-      <origin xyz="-15.0 -6.0 -1.0" rpy="0 0 0"/>
+      <origin xyz="15.0 -6.0 -1.0" rpy="0 0 0"/>
     </joint>
     <!-- Robot world origin -->
