Commit message: update rviz file

File: description/xacro/robot_system_multi_interface.urdf.xacro (robot description, xacro)
@@ -68,7 +68,8 @@
   <xacro:instantiate_robots index="0" count="${int(sim_robot_count)}"/>
   <xacro:if value="${use_manipulator_hardware or use_vehicle_hardware}">
+    <xacro:property name="prefix" value="robot_real_"/>
     <!-- Instantiate the real robot -->
     <xacro:bluerov2_heavy_alpha_urdf
-      prefix="real_"
+      prefix="${prefix}"
       x="0.0"
       y="0.0"
@@ -79,5 +80,5 @@
     <xacro:robot_system_multi_interface
       name="$real_ReachSystemMultiInterface"
-      prefix="real_"
+      prefix="${prefix}"
       serial_port="${serial_port}"
       state_update_frequency="${state_update_frequency}"
@@ -85,10 +86,10 @@
     <xacro:vehicle_system_multi_interface
       name="real_BlueSystemMultiInterface"
-      prefix="real_"
+      prefix="${prefix}"
       serial_port="${serial_port}"
       state_update_frequency="${state_update_frequency}"
       use_hardware="${use_vehicle_hardware}"
       frame_id="base_link"
-      child_frame_id="real_base_link"/>
+      child_frame_id="${prefix}base_link"/>
   </xacro:if>
 </robot>

Commit message: fix ned frame as map

File: description/xacro/robot_system_multi_interface.urdf.xacro (robot description, xacro)
@@ -59,5 +59,5 @@
       state_update_frequency="${state_update_frequency}"
       use_hardware="false"
-      frame_id="base_link"
+      frame_id="ned_frame"
       child_frame_id="${prefix}base_link"/>
       <!-- Recursively call the macro for the next robot -->
@@ -90,5 +90,5 @@
       state_update_frequency="${state_update_frequency}"
       use_hardware="${use_vehicle_hardware}"
-      frame_id="base_link"
+      frame_id="ned_frame"
       child_frame_id="${prefix}base_link"/>
   </xacro:if>

File: description/xacro/urdf.xacro (robot description, xacro)
@@ -59,5 +59,5 @@
     <joint name="${prefix}base_joint" type="fixed">
       <child link="${prefix}base_link" />
-      <parent link="base_link" />
+      <parent link="ned_frame" />
       <origin xyz="${x} ${y} ${z}" rpy="${rot_r} ${rot_p} ${rot_y}"/>
     </joint>

File: description/xacro/world.xacro (robot description, xacro)
@@ -68,4 +68,11 @@
       <origin xyz="0.0 0.0 0.0" rpy="0 0 0"/>
     </joint>
+    <!-- Robot NED origin -->
+    <link name="ned_frame"/>
+    <joint name="ned_frame_joint" type="fixed">
+      <child link="ned_frame" />
+      <parent link="world" />
+      <origin xyz="0.0 0.0 0.0" rpy="3.14159265359 0 0"/>
+    </joint>
   </xacro:macro>
 </robot>
