Commit message: added sea floor

File: description/xacro/urdf.xacro (robot description, xacro)
@@ -12,14 +12,26 @@
     </link>
     <link name="world_bottom"/>
-    <joint name="world_bottom_joint" type="fixed">
-      <child link="world_bottom" />
-      <parent link="world" />
-      <origin xyz="0.0 0.0 -6.0" rpy="0 0 0"/>
-    </joint>
-  <link name="bathymetry">
+    <link name="bathymetry_shipwreck">
       <visual>
         <origin xyz="0 0 0" rpy="${pi/2} 0 0"/>
         <geometry>
-          <mesh filename="file://$(find ros2_control_blue_reach_5)/Bathymetry/meshes/Manhomansett.stl"/>
+          <mesh filename="file://$(find ros2_control_blue_reach_5)/Bathymetry/meshes/Manhomansett.stl" scale="5 5 5"/>
+        </geometry>
+        <material name="gray">
+          <color rgba="0.5 0.5 0.5 1.0"/>
+        </material>
+      </visual>
+      <collision>
+        <origin xyz="0 0 0" rpy="${pi/2} 0 0"/>
+        <geometry>
+          <mesh filename="file://$(find ros2_control_blue_reach_5)/Bathymetry/meshes/Manhomansett.stl" scale="5 5 5"/>
+        </geometry>
+      </collision>
+    </link>
+    <link name="bathymetry_seafloor">
+      <visual>
+        <origin xyz="0 0 0" rpy="0 0 0"/>
+        <geometry>
+          <mesh filename="file://$(find ros2_control_blue_reach_5)/Bathymetry/meshes/hawaii.stl" scale="0.4 0.4 0.4"/>
         </geometry>
         <material name="gray">
@@ -30,12 +42,22 @@
         <origin xyz="0 0 0" rpy="0 0 0"/>
         <geometry>
-          <mesh filename="file://$(find ros2_control_blue_reach_5)/Bathymetry/meshes/Manhomansett.stl"/>
+          <mesh filename="file://$(find ros2_control_blue_reach_5)/Bathymetry/meshes/hawaii.stl" scale="0.4 0.4 0.4"/>
         </geometry>
       </collision>
     </link>
-    <joint name="bathymetry_joint" type="fixed">
-      <child link="bathymetry" />
+    <joint name="world_bottom_joint" type="fixed">
+      <child link="world_bottom" />
+      <parent link="world" />
+      <origin xyz="0.0 0.0 -8.0" rpy="0 0 0"/>
+    </joint>
+    <joint name="bathymetry_seafloor_joint" type="fixed">
+      <child link="bathymetry_seafloor" />
       <parent link="world_bottom" />
-      <origin xyz="0.0 0.0 -0.3" rpy="0 0 0"/>
+      <origin xyz="0.0 0.0 0.0" rpy="0 0 0"/>
+    </joint>
+   <joint name="bathymetry_shipwreck_joint" type="fixed">
+      <child link="bathymetry_shipwreck" />
+      <parent link="bathymetry_seafloor" />
+      <origin xyz="-15.0 -6.0 -1.0" rpy="0 0 0"/>
     </joint>
     <!-- Robot body origin -->

Commit message: added sea floor

File: description/xacro/urdf.xacro (robot description, xacro)
@@ -52,5 +52,5 @@
     </joint>
     <joint name="bathymetry_seafloor_joint" type="fixed">
-      <child link="bathymetry_seafloor" />
+      <child link="bathymetry_seafloor"/>
       <parent link="world_bottom" />
       <origin xyz="0.0 0.0 0.0" rpy="0 0 0"/>

Commit message: clean up

File: description/xacro/urdf.xacro (robot description, xacro)
@@ -16,5 +16,5 @@
         <origin xyz="0 0 0" rpy="${pi/2} 0 0"/>
         <geometry>
-          <mesh filename="file://$(find ros2_control_blue_reach_5)/Bathymetry/meshes/Manhomansett.stl" scale="5 5 5"/>
+          <mesh filename="file://$(find ros2_control_blue_reach_5)/Bathymetry/meshes/manhomansett.stl" scale="5 5 5"/>
         </geometry>
         <material name="gray">
@@ -25,9 +25,9 @@
         <origin xyz="0 0 0" rpy="${pi/2} 0 0"/>
         <geometry>
-          <mesh filename="file://$(find ros2_control_blue_reach_5)/Bathymetry/meshes/Manhomansett.stl" scale="5 5 5"/>
+          <mesh filename="file://$(find ros2_control_blue_reach_5)/Bathymetry/meshes/manhomansett.stl" scale="5 5 5"/>
         </geometry>
       </collision>
     </link>
-    <link name="bathymetry_seafloor">
+    <!-- <link name="bathymetry_seafloor">
       <visual>
         <origin xyz="0 0 0" rpy="0 0 0"/>
@@ -45,5 +45,5 @@
         </geometry>
       </collision>
-    </link>
+    </link> -->
     <joint name="world_bottom_joint" type="fixed">
       <child link="world_bottom" />
@@ -51,12 +51,12 @@
       <origin xyz="0.0 0.0 -8.0" rpy="0 0 0"/>
     </joint>
-    <joint name="bathymetry_seafloor_joint" type="fixed">
+    <!-- <joint name="bathymetry_seafloor_joint" type="fixed">
       <child link="bathymetry_seafloor"/>
       <parent link="world_bottom" />
       <origin xyz="0.0 0.0 0.0" rpy="0 0 0"/>
-    </joint>
+    </joint> -->
    <joint name="bathymetry_shipwreck_joint" type="fixed">
       <child link="bathymetry_shipwreck" />
-      <parent link="bathymetry_seafloor" />
+      <parent link="world_bottom" />
       <origin xyz="-15.0 -6.0 -1.0" rpy="0 0 0"/>
     </joint>

Commit message: testing robot localization

File: description/xacro/urdf.xacro (robot description, xacro)
@@ -62,4 +62,11 @@
       <origin xyz="${x} ${y} ${z}" rpy="${rot_r} ${rot_p} ${rot_y}"/>
     </joint>
+    <!-- Robot body NED -->
+    <link name="${prefix}body_ned"/>
+    <joint name="${prefix}body_ned_joint" type="fixed">
+      <child link="${prefix}body_ned" />
+      <parent link="${prefix}base_link" />
+      <origin xyz="0.0 0.0 0.0" rpy="${pi} 0 0"/>
+    </joint>
     <joint name="${prefix}manipulator_mount_joint" type="fixed">
       <origin rpy="0 0 0" xyz="0.14 0.0 -0.12" />

File: description/xacro/world.xacro (robot description, xacro)
@@ -73,5 +73,5 @@
       <child link="ned_frame" />
       <parent link="world" />
-      <origin xyz="0.0 0.0 0.0" rpy="3.14159265359 0 0"/>
+      <origin xyz="0.0 0.0 0.0" rpy="${pi} 0 0"/>
     </joint>
   </xacro:macro>
