Commit message: bathymetry added

File: description/ros2_control/robot_system_multi_interface.ros2_control.xacro (robot description, xacro)
@@ -6,5 +6,5 @@
       <hardware>
         <xacro:if value="${use_mock_hardware}">
-          <plugin>ros2_control_blue_reach_5/RRBotSystemMultiInterfaceHardware</plugin>
+          <plugin>ros2_control_blue_reach_5/SimReachSystemMultiInterfaceHardware</plugin>
           <param name="state_update_frequency">${state_update_frequency}</param>
         </xacro:if>

File: description/xacro/urdf.xacro (robot description, xacro)
@@ -16,4 +16,26 @@
       <parent link="world" />
       <origin xyz="0.0 0.0 -6.0" rpy="0 0 0"/>
+    </joint>
+  <link name="bathymetry">
+      <visual>
+        <origin xyz="0 0 0" rpy="${pi/2} 0 0"/>
+        <geometry>
+          <mesh filename="file://$(find ros2_control_blue_reach_5)/Bathymetry/meshes/Manhomansett.stl"/>
+        </geometry>
+        <material name="gray">
+          <color rgba="0.5 0.5 0.5 1.0"/>
+        </material>
+      </visual>
+      <collision>
+        <origin xyz="0 0 0" rpy="0 0 0"/>
+        <geometry>
+          <mesh filename="file://$(find ros2_control_blue_reach_5)/Bathymetry/meshes/Manhomansett.stl"/>
+        </geometry>
+      </collision>
+    </link>
+    <joint name="bathymetry_joint" type="fixed">
+      <child link="bathymetry" />
+      <parent link="world_bottom" />
+      <origin xyz="0.0 0.0 -0.3" rpy="0 0 0"/>
     </joint>
     <!-- Robot body origin -->

Commit message: update

File: description/ros2_control/robot_system_multi_interface.ros2_control.xacro (robot description, xacro)
@@ -15,58 +15,164 @@
         </xacro:unless>
       </hardware>
-      <joint name="${prefix}_axis_a">
-        <param name="device_id">0x01</param>
-        <param name="home">0.0</param>
-        <!-- limit constraints -->
-        <param name="max_effort">200</param>
-        <param name="has_position_limits">1</param>
-        <param name="min_position">0.0004</param>
-        <param name="max_position">0.0137</param>
-        <param name="max_velocity">3.0</param>
-        <param name="soft_k_position">100</param>
-        <param name="soft_k_velocity">10</param>
-        <param name="soft_min_position">0.0004</param>
-        <param name="soft_max_position">0.0137</param>
-        <param name="kt">50</param>  <!-- static friction current -->
-        <param name="forward_I_static">43</param> <!-- static friction torque -->
-        <param name="backward_I_static">43</param> <!-- static friction torque -->
-        <!-- limit constraints -->
-          <command_interface name="position">
-            <param name="min">-1</param>
-            <param name="max">1</param>
-          </command_interface>
-          <command_interface name="velocity">
-            <param name="min">-1</param>
-            <param name="max">1</param>
-          </command_interface>
-          <command_interface name="current">
-            <param name="min">-1</param>
-            <param name="max">1</param>
-          </command_interface>
-          <command_interface name="effort">
-            <param name="min">-1</param>
-            <param name="max">1</param>
-          </command_interface>
-        <state_interface name="position"/>
-        <state_interface name="filtered_position"/>
-        <state_interface name="velocity"/>
-        <state_interface name="filtered_velocity"/>
-        <state_interface name="acceleration"/>
-        <state_interface name="estimated_acceleration"/>
-        <state_interface name="current"/>
-        <state_interface name="effort"/>
-        <state_interface name="computed_effort"/>
-        <state_interface name="computed_effort_uncertainty"/>
-        <state_interface name="predicted_position"/>
-        <state_interface name="predicted_position_uncertainty"/>
-        <state_interface name="predicted_velocity"/>
-        <state_interface name="predicted_velocity_uncertainty"/>
-        <state_interface name="adaptive_predicted_position"/>
-        <state_interface name="adaptive_predicted_position_uncertainty"/>
-        <state_interface name="adaptive_predicted_velocity"/>
-        <state_interface name="adaptive_predicted_velocity_uncertainty"/>
-        <state_interface name="stateId"/>
-      </joint>
-      <joint name="${prefix}_axis_b">
+      <joint name="${prefix}_axis_e">
+        <param name="device_id">0x05</param>
+        <param name="home">1.92466658e-02</param>
+        <!-- limit constraints -->
+        <param name="max_effort">300</param>
+        <param name="has_position_limits">1</param>
+        <param name="min_position">1.0</param>
+        <param name="max_position">5.5</param>
+        <param name="max_velocity">4.0</param>
+        <param name="soft_k_position">100</param>
+        <param name="soft_k_velocity">10</param>
+        <param name="soft_min_position">1.0</param>
+        <param name="soft_max_position">5.5</param>
+        <param name="kt">90.6</param>  <!-- static friction current -->
+        <param name="forward_I_static">43</param> <!-- static friction torque -->
+        <param name="backward_I_static">43</param> <!-- static friction torque -->
+        <!-- limit constraints -->
+          <command_interface name="position">
+            <param name="min">-1</param>
+            <param name="max">1</param>
+          </command_interface>
+          <command_interface name="velocity">
+            <param name="min">-1</param>
+            <param name="max">1</param>
+          </command_interface>
+          <command_interface name="current">
+            <param name="min">-1</param>
+            <param name="max">1</param>
+          </command_interface>
+          <command_interface name="effort">
+            <param name="min">-1</param>
+            <param name="max">1</param>
+          </command_interface>
+        <state_interface name="position"/>
+        <state_interface name="filtered_position"/>
+        <state_interface name="velocity"/>
+        <state_interface name="filtered_velocity"/>
+        <state_interface name="acceleration"/>
+        <state_interface name="estimated_acceleration"/>
+        <state_interface name="current"/>
+        <state_interface name="effort"/>
+        <state_interface name="computed_effort"/>
+        <state_interface name="computed_effort_uncertainty"/>
+        <state_interface name="predicted_position"/>
+        <state_interface name="predicted_position_uncertainty"/>
+        <state_interface name="predicted_velocity"/>
+        <state_interface name="predicted_velocity_uncertainty"/>
+        <state_interface name="adaptive_predicted_position"/>
+        <state_interface name="adaptive_predicted_position_uncertainty"/>
+        <state_interface name="adaptive_predicted_velocity"/>
+        <state_interface name="adaptive_predicted_velocity_uncertainty"/>
+        <state_interface name="stateId"/>
+      </joint>
+    <joint name="${prefix}_axis_d">
+        <param name="device_id">0x04</param>
+        <param name="home">1.45291960e+00</param>
+        <!-- limit constraints -->
+        <param name="max_effort">200</param>
+        <param name="has_position_limits">1</param>
+        <param name="min_position">0.01</param>
+        <param name="max_position">3.400</param>
+        <param name="max_velocity">4.0</param>
+        <param name="soft_k_position">100</param>
+        <param name="soft_k_velocity">10</param>
+        <param name="soft_min_position">0.01</param>
+        <param name="soft_max_position">3.400</param>
+        <param name="kt">90.6</param>  <!-- static friction current -->
+        <param name="forward_I_static">43</param> <!-- static friction torque -->
+        <param name="backward_I_static">43</param> <!-- static friction torque -->
+        <!-- limit constraints -->
+          <command_interface name="position">
+            <param name="min">-1</param>
+            <param name="max">1</param>
+          </command_interface>
+          <command_interface name="velocity">
+            <param name="min">-1</param>
+            <param name="max">1</param>
+          </command_interface>
+          <command_interface name="current">
+            <param name="min">-1</param>
+            <param name="max">1</param>
+          </command_interface>
+          <command_interface name="effort">
+            <param name="min">-1</param>
+            <param name="max">1</param>
+          </command_interface>
+        <state_interface name="position"/>
+        <state_interface name="filtered_position"/>
+        <state_interface name="velocity"/>
+        <state_interface name="filtered_velocity"/>
+        <state_interface name="acceleration"/>
+        <state_interface name="estimated_acceleration"/>
+        <state_interface name="current"/>
+        <state_interface name="effort"/>
+        <state_interface name="computed_effort"/>
+        <state_interface name="computed_effort_uncertainty"/>
+        <state_interface name="predicted_position"/>
+        <state_interface name="predicted_position_uncertainty"/>
+        <state_interface name="predicted_velocity"/>
+        <state_interface name="predicted_velocity_uncertainty"/>
+        <state_interface name="adaptive_predicted_position"/>
+        <state_interface name="adaptive_predicted_position_uncertainty"/>
+        <state_interface name="adaptive_predicted_velocity"/>
+        <state_interface name="adaptive_predicted_velocity_uncertainty"/>
+        <state_interface name="stateId"/>
+      </joint>
+      <joint name="${prefix}_axis_c">
+        <param name="device_id">0x03</param>
+        <param name="home">4.35027387e-03</param>
+        <!-- limit constraints -->
+        <param name="max_effort">200</param>
+        <param name="has_position_limits">1</param>
+        <param name="min_position">0.01</param>
+        <param name="max_position">3.400</param>
+        <param name="max_velocity">4.0</param>
+        <param name="soft_k_position">100</param>
+        <param name="soft_k_velocity">10</param>
+        <param name="soft_min_position">0.01</param>
+        <param name="soft_max_position">3.400</param>
+        <param name="kt">90.6</param>  <!-- static friction current -->
+        <param name="forward_I_static">43</param> <!-- static friction torque -->
+        <param name="backward_I_static">43</param> <!-- static friction torque -->
+        <!-- limit constraints -->
+          <command_interface name="position">
+            <param name="min">-1</param>
+            <param name="max">1</param>
+          </command_interface>
+          <command_interface name="velocity">
+            <param name="min">-1</param>
+            <param name="max">1</param>
+          </command_interface>
+          <command_interface name="current">
+            <param name="min">-1</param>
+            <param name="max">1</param>
+          </command_interface>
+          <command_interface name="effort">
+            <param name="min">-1</param>
+            <param name="max">1</param>
+          </command_interface>
+        <state_interface name="position"/>
+        <state_interface name="filtered_position"/>
+        <state_interface name="velocity"/>
+        <state_interface name="filtered_velocity"/>
+        <state_interface name="acceleration"/>
+        <state_interface name="estimated_acceleration"/>
+        <state_interface name="current"/>
+        <state_interface name="effort"/>
+        <state_interface name="computed_effort"/>
+        <state_interface name="computed_effort_uncertainty"/>
+        <state_interface name="predicted_position"/>
+        <state_interface name="predicted_position_uncertainty"/>
+        <state_interface name="predicted_velocity"/>
+        <state_interface name="predicted_velocity_uncertainty"/>
+        <state_interface name="adaptive_predicted_position"/>
+        <state_interface name="adaptive_predicted_position_uncertainty"/>
+        <state_interface name="adaptive_predicted_velocity"/>
+        <state_interface name="adaptive_predicted_velocity_uncertainty"/>
+        <state_interface name="stateId"/>
+      </joint>
+  <joint name="${prefix}_axis_b">
         <param name="device_id">0x02</param>
         <param name="home">5.690</param>
@@ -121,124 +227,18 @@
         <state_interface name="stateId"/>
       </joint>
-      <joint name="${prefix}_axis_c">
-        <param name="device_id">0x03</param>
-        <param name="home">4.35027387e-03</param>
-        <!-- limit constraints -->
-        <param name="max_effort">200</param>
-        <param name="has_position_limits">1</param>
-        <param name="min_position">0.01</param>
-        <param name="max_position">3.400</param>
-        <param name="max_velocity">4.0</param>
-        <param name="soft_k_position">100</param>
-        <param name="soft_k_velocity">10</param>
-        <param name="soft_min_position">0.01</param>
-        <param name="soft_max_position">3.400</param>
-        <param name="kt">90.6</param>  <!-- static friction current -->
-        <param name="forward_I_static">43</param> <!-- static friction torque -->
-        <param name="backward_I_static">43</param> <!-- static friction torque -->
-        <!-- limit constraints -->
-          <command_interface name="position">
-            <param name="min">-1</param>
-            <param name="max">1</param>
-          </command_interface>
-          <command_interface name="velocity">
-            <param name="min">-1</param>
-            <param name="max">1</param>
-          </command_interface>
-          <command_interface name="current">
-            <param name="min">-1</param>
-            <param name="max">1</param>
-          </command_interface>
-          <command_interface name="effort">
-            <param name="min">-1</param>
-            <param name="max">1</param>
-          </command_interface>
-        <state_interface name="position"/>
-        <state_interface name="filtered_position"/>
-        <state_interface name="velocity"/>
-        <state_interface name="filtered_velocity"/>
-        <state_interface name="acceleration"/>
-        <state_interface name="estimated_acceleration"/>
-        <state_interface name="current"/>
-        <state_interface name="effort"/>
-        <state_interface name="computed_effort"/>
-        <state_interface name="computed_effort_uncertainty"/>
-        <state_interface name="predicted_position"/>
-        <state_interface name="predicted_position_uncertainty"/>
-        <state_interface name="predicted_velocity"/>
-        <state_interface name="predicted_velocity_uncertainty"/>
-        <state_interface name="adaptive_predicted_position"/>
-        <state_interface name="adaptive_predicted_position_uncertainty"/>
-        <state_interface name="adaptive_predicted_velocity"/>
-        <state_interface name="adaptive_predicted_velocity_uncertainty"/>
-        <state_interface name="stateId"/>
-      </joint>
-      <joint name="${prefix}_axis_d">
-        <param name="device_id">0x04</param>
-        <param name="home">1.45291960e+00</param>
-        <!-- limit constraints -->
-        <param name="max_effort">200</param>
-        <param name="has_position_limits">1</param>
-        <param name="min_position">0.01</param>
-        <param name="max_position">3.400</param>
-        <param name="max_velocity">4.0</param>
-        <param name="soft_k_position">100</param>
-        <param name="soft_k_velocity">10</param>
-        <param name="soft_min_position">0.01</param>
-        <param name="soft_max_position">3.400</param>
-        <param name="kt">90.6</param>  <!-- static friction current -->
-        <param name="forward_I_static">43</param> <!-- static friction torque -->
-        <param name="backward_I_static">43</param> <!-- static friction torque -->
-        <!-- limit constraints -->
-          <command_interface name="position">
-            <param name="min">-1</param>
-            <param name="max">1</param>
-          </command_interface>
-          <command_interface name="velocity">
-            <param name="min">-1</param>
-            <param name="max">1</param>
-          </command_interface>
-          <command_interface name="current">
-            <param name="min">-1</param>
-            <param name="max">1</param>
-          </command_interface>
-          <command_interface name="effort">
-            <param name="min">-1</param>
-            <param name="max">1</param>
-          </command_interface>
-        <state_interface name="position"/>
-        <state_interface name="filtered_position"/>
-        <state_interface name="velocity"/>
-        <state_interface name="filtered_velocity"/>
-        <state_interface name="acceleration"/>
-        <state_interface name="estimated_acceleration"/>
-        <state_interface name="current"/>
-        <state_interface name="effort"/>
-        <state_interface name="computed_effort"/>
-        <state_interface name="computed_effort_uncertainty"/>
-        <state_interface name="predicted_position"/>
-        <state_interface name="predicted_position_uncertainty"/>
-        <state_interface name="predicted_velocity"/>
-        <state_interface name="predicted_velocity_uncertainty"/>
-        <state_interface name="adaptive_predicted_position"/>
-        <state_interface name="adaptive_predicted_position_uncertainty"/>
-        <state_interface name="adaptive_predicted_velocity"/>
-        <state_interface name="adaptive_predicted_velocity_uncertainty"/>
-        <state_interface name="stateId"/>
-      </joint>
-      <joint name="${prefix}_axis_e">
-        <param name="device_id">0x05</param>
-        <param name="home">1.92466658e-02</param>
-        <!-- limit constraints -->
-        <param name="max_effort">300</param>
-        <param name="has_position_limits">1</param>
-        <param name="min_position">1.0</param>
-        <param name="max_position">5.5</param>
-        <param name="max_velocity">4.0</param>
-        <param name="soft_k_position">100</param>
-        <param name="soft_k_velocity">10</param>
-        <param name="soft_min_position">1.0</param>
-        <param name="soft_max_position">5.5</param>
-        <param name="kt">90.6</param>  <!-- static friction current -->
+      <joint name="${prefix}_axis_a">
+        <param name="device_id">0x01</param>
+        <param name="home">0.0</param>
+        <!-- limit constraints -->
+        <param name="max_effort">200</param>
+        <param name="has_position_limits">1</param>
+        <param name="min_position">0.0004</param>
+        <param name="max_position">0.0137</param>
+        <param name="max_velocity">3.0</param>
+        <param name="soft_k_position">100</param>
+        <param name="soft_k_velocity">10</param>
+        <param name="soft_min_position">0.0004</param>
+        <param name="soft_max_position">0.0137</param>
+        <param name="kt">50</param>  <!-- static friction current -->
         <param name="forward_I_static">43</param> <!-- static friction torque -->
         <param name="backward_I_static">43</param> <!-- static friction torque -->
