Commit message: update docs

File: description/ros2_control/robot_system_multi_interface.ros2_control.xacro (robot description, xacro)
@@ -2,14 +2,14 @@
 <robot xmlns:xacro="http://www.ros.org/wiki/xacro">
   <xacro:macro name="robot_system_multi_interface"
-  params="name prefix serial_port state_update_frequency use_mock_hardware">
+  params="name prefix serial_port state_update_frequency use_hardware">
     <ros2_control name="${name}" type="system">
       <hardware>
-        <xacro:if value="${use_mock_hardware}">
-          <plugin>ros2_control_blue_reach_5/SimReachSystemMultiInterfaceHardware</plugin>
+        <xacro:if value="${use_hardware}">
+          <plugin>ros2_control_blue_reach_5/ReachSystemMultiInterfaceHardware</plugin>
+          <param name="serial_port">${serial_port}</param>
           <param name="state_update_frequency">${state_update_frequency}</param>
         </xacro:if>
-        <xacro:unless value="${use_mock_hardware}">
-          <plugin>ros2_control_blue_reach_5/ReachSystemMultiInterfaceHardware</plugin>
-          <param name="serial_port">${serial_port}</param>
+        <xacro:unless value="${use_hardware}">
+          <plugin>ros2_control_blue_reach_5/SimReachSystemMultiInterfaceHardware</plugin>
           <param name="state_update_frequency">${state_update_frequency}</param>
         </xacro:unless>

File: description/ros2_control/vehicle_system_multi_interface.ros2_control.xacro (robot description, xacro)
@@ -1,8 +1,8 @@
 <?xml version="1.0"?>
 <robot xmlns:xacro="http://www.ros.org/wiki/xacro">
-  <xacro:macro name="vehicle_system_multi_interface" params="name prefix serial_port state_update_frequency use_mock_hardware frame_id child_frame_id">
+  <xacro:macro name="vehicle_system_multi_interface" params="name prefix serial_port state_update_frequency use_hardware frame_id child_frame_id">
     <ros2_control name="${name}" type="system">
       <hardware>
-        <xacro:if value="${use_mock_hardware}">
+        <xacro:if value="${use_hardware}">
           <plugin>ros2_control_blue_reach_5/SimVehicleSystemMultiInterfaceHardware</plugin>
           <param name="prefix">${prefix}</param>
@@ -10,6 +10,9 @@
           <param name="child_frame_id">${child_frame_id}</param>
         </xacro:if>
-        <xacro:unless value="${use_mock_hardware}">
-          <plugin>ros2_control_blue_reach_5/VehicleSystemMultiInterfaceHardware</plugin>
+        <xacro:unless value="${use_hardware}">
+          <plugin>ros2_control_blue_reach_5/SimVehicleSystemMultiInterfaceHardware</plugin>
+          <param name="prefix">${prefix}</param>
+          <param name="frame_id">${frame_id}</param>
+          <param name="child_frame_id">${child_frame_id}</param>
         </xacro:unless>
       </hardware>

File: description/xacro/robot_system_multi_interface.urdf.xacro (robot description, xacro)
@@ -2,6 +2,7 @@
 <robot xmlns:xacro="http://www.ros.org/wiki/xacro" name="alpha_5_example">
   <!-- Enable setting arguments from the launch file -->
-  <xacro:arg name="use_mock_hardware" default="true"/>
-  <xacro:arg name="robot_count" default="4"/>
+  <xacro:arg name="use_manipulator_hardware" default="false"/>
+  <xacro:arg name="use_vehicle_hardware" default="false"/>
+  <xacro:arg name="sim_robot_count" default="4"/>
   <xacro:arg name="serial_port" default="/dev/ttyUSB0"/>
   <xacro:arg name="state_update_frequency" default="250"/>
@@ -9,8 +10,9 @@
   <!-- Properties -->
   <xacro:property name="description_package" value="$(arg description_package)"/>
-  <xacro:property name="robot_count" value="$(arg robot_count)"/>
+  <xacro:property name="sim_robot_count" value="$(arg sim_robot_count)"/>
   <xacro:property name="serial_port" value="$(arg serial_port)"/>
   <xacro:property name="state_update_frequency" value="$(arg state_update_frequency)"/>
-  <xacro:property name="use_mock_hardware" value="$(arg use_mock_hardware)"/>
+  <xacro:property name="use_manipulator_hardware" value="$(arg use_manipulator_hardware)"/>
+  <xacro:property name="use_vehicle_hardware" value="$(arg use_vehicle_hardware)"/>
   <!-- Define constants -->
   <xacro:property name="d_min" value="1.0"/>
@@ -50,5 +52,5 @@
       serial_port="${serial_port}"
       state_update_frequency="${state_update_frequency}"
-      use_mock_hardware="${use_mock_hardware}"/>
+      use_hardware="false"/>
     <xacro:vehicle_system_multi_interface
       name="${prefix}BlueSystemMultiInterface"
@@ -56,5 +58,5 @@
       serial_port="${serial_port}"
       state_update_frequency="${state_update_frequency}"
-      use_mock_hardware="${use_mock_hardware}"
+      use_hardware="false"
       frame_id="base_link"
       child_frame_id="${prefix}base_link"/>
@@ -64,27 +66,29 @@
   </xacro:macro>
   <!-- Start the robot instantiation recursion -->
-  <xacro:instantiate_robots index="0" count="${int(robot_count)}"/>
-  <!-- Instantiate the real robot -->
-  <xacro:bluerov2_heavy_alpha_urdf
-    prefix="real_"
-    x="0.0"
-    y="0.0"
-    z="0.0"
-    rot_r="0.0"
-    rot_p="0.0"
-    rot_y="0.0"/>
-  <xacro:robot_system_multi_interface
-    name="$real_ReachSystemMultiInterface"
-    prefix="real_"
-    serial_port="${serial_port}"
-    state_update_frequency="${state_update_frequency}"
-    use_mock_hardware="false"/>
-  <xacro:vehicle_system_multi_interface
-    name="real_BlueSystemMultiInterface"
-    prefix="real_"
-    serial_port="${serial_port}"
-    state_update_frequency="${state_update_frequency}"
-    use_mock_hardware="${use_mock_hardware}"
-    frame_id="base_link"
-    child_frame_id="real_base_link"/>
+  <xacro:instantiate_robots index="0" count="${int(sim_robot_count)}"/>
+  <xacro:if value="${use_manipulator_hardware or use_vehicle_hardware}">
+    <!-- Instantiate the real robot -->
+    <xacro:bluerov2_heavy_alpha_urdf
+      prefix="real_"
+      x="0.0"
+      y="0.0"
+      z="0.0"
+      rot_r="0.0"
+      rot_p="0.0"
+      rot_y="0.0"/>
+    <xacro:robot_system_multi_interface
+      name="$real_ReachSystemMultiInterface"
+      prefix="real_"
+      serial_port="${serial_port}"
+      state_update_frequency="${state_update_frequency}"
+      use_hardware="${use_manipulator_hardware}"/>
+    <xacro:vehicle_system_multi_interface
+      name="real_BlueSystemMultiInterface"
+      prefix="real_"
+      serial_port="${serial_port}"
+      state_update_frequency="${state_update_frequency}"
+      use_hardware="${use_vehicle_hardware}"
+      frame_id="base_link"
+      child_frame_id="real_base_link"/>
+  </xacro:if>
 </robot>
