Commit message: multiagent supported

File: description/ros2_control/vehicle_system_multi_interface.ros2_control.xacro (robot description, xacro)
@@ -1,10 +1,12 @@
 <?xml version="1.0"?>
 <robot xmlns:xacro="http://www.ros.org/wiki/xacro">
-  <xacro:macro name="vehicle_system_multi_interface"
-  params="name prefix serial_port state_update_frequency use_mock_hardware">
+  <xacro:macro name="vehicle_system_multi_interface" params="name prefix serial_port state_update_frequency use_mock_hardware frame_id child_frame_id">
     <ros2_control name="${name}" type="system">
       <hardware>
         <xacro:if value="${use_mock_hardware}">
           <plugin>ros2_control_blue_reach_5/SimVehicleSystemMultiInterfaceHardware</plugin>
+          <param name="prefix">${prefix}</param>
+          <param name="frame_id">${frame_id}</param>
+          <param name="child_frame_id">${child_frame_id}</param>
         </xacro:if>
         <xacro:unless value="${use_mock_hardware}">

File: description/xacro/robot_system_multi_interface.urdf.xacro (robot description, xacro)
@@ -3,5 +3,5 @@
   <!-- Enable setting arguments from the launch file -->
   <xacro:arg name="use_mock_hardware" default="true"/>
-  <xacro:arg name="robot_count" default="1"/>
+  <xacro:arg name="robot_count" default="4"/>
   <xacro:arg name="serial_port" default="/dev/ttyUSB0"/>
   <xacro:arg name="state_update_frequency" default="250"/>
@@ -46,5 +46,5 @@
         rot_y="${angle}"/>
     <xacro:robot_system_multi_interface
-      name="ReachSystemMultiInterface"
+      name="${prefix}ReachSystemMultiInterface"
       prefix="${prefix}"
       serial_port="${serial_port}"
@@ -52,9 +52,11 @@
       use_mock_hardware="${use_mock_hardware}"/>
     <xacro:vehicle_system_multi_interface
-      name="BlueSystemMultiInterface"
+      name="${prefix}BlueSystemMultiInterface"
       prefix="${prefix}"
       serial_port="${serial_port}"
       state_update_frequency="${state_update_frequency}"
-      use_mock_hardware="${use_mock_hardware}"/>
+      use_mock_hardware="${use_mock_hardware}"
+      frame_id="base_link"
+      child_frame_id="${prefix}base_link"/>
       <!-- Recursively call the macro for the next robot -->
       <xacro:instantiate_robots index="${index + 1}" count="${count}"/>

Commit message: update hil

File: description/ros2_control/vehicle_system_multi_interface.ros2_control.xacro (robot description, xacro)
@@ -1,5 +1,5 @@
 <?xml version="1.0"?>
 <robot xmlns:xacro="http://www.ros.org/wiki/xacro">
-  <xacro:macro name="vehicle_system_multi_interface" params="name prefix serial_port state_update_frequency use_hardware frame_id child_frame_id">
+  <xacro:macro name="vehicle_system_multi_interface" params="name prefix serial_port state_update_frequency use_hardware frame_id child_frame_id map_frame_id">
     <ros2_control name="${name}" type="system">
       <hardware>
@@ -9,4 +9,5 @@
           <param name="frame_id">${frame_id}</param>
           <param name="child_frame_id">${child_frame_id}</param>
+          <param name="map_frame_id">${map_frame_id}</param>
         </xacro:if>
         <xacro:unless value="${use_hardware}">
@@ -15,4 +16,5 @@
           <param name="frame_id">${frame_id}</param>
           <param name="child_frame_id">${child_frame_id}</param>
+          <param name="map_frame_id">${map_frame_id}</param>
         </xacro:unless>
       </hardware>

File: description/xacro/robot_system_multi_interface.urdf.xacro (robot description, xacro)
@@ -59,6 +59,7 @@
       state_update_frequency="${state_update_frequency}"
       use_hardware="false"
-      frame_id="ned_frame"
-      child_frame_id="${prefix}base_link"/>
+      frame_id="base_link"
+      child_frame_id="${prefix}base_link"
+      map_frame_id="${prefix}map"/>
       <!-- Recursively call the macro for the next robot -->
       <xacro:instantiate_robots index="${index + 1}" count="${count}"/>
@@ -90,6 +91,7 @@
       state_update_frequency="${state_update_frequency}"
       use_hardware="${use_vehicle_hardware}"
-      frame_id="ned_frame"
-      child_frame_id="${prefix}base_link"/>
+      frame_id="base_link"
+      child_frame_id="${prefix}base_link"
+      map_frame_id="${prefix}map"/>
   </xacro:if>
 </robot>

File: description/xacro/urdf.xacro (robot description, xacro)
@@ -59,13 +59,6 @@
     <joint name="${prefix}base_joint" type="fixed">
       <child link="${prefix}base_link" />
-      <parent link="ned_frame" />
+      <parent link="base_link" />
       <origin xyz="${x} ${y} ${z}" rpy="${rot_r} ${rot_p} ${rot_y}"/>
-    </joint>
-    <!-- Robot body NED -->
-    <link name="${prefix}body_ned"/>
-    <joint name="${prefix}body_ned_joint" type="fixed">
-      <child link="${prefix}body_ned" />
-      <parent link="${prefix}base_link" />
-      <origin xyz="0.0 0.0 0.0" rpy="${pi} 0 0"/>
     </joint>
     <joint name="${prefix}manipulator_mount_joint" type="fixed">

File: description/xacro/world.xacro (robot description, xacro)
@@ -68,11 +68,4 @@
       <origin xyz="0.0 0.0 0.0" rpy="0 0 0"/>
     </joint>
-    <!-- Robot NED origin -->
-    <link name="ned_frame"/>
-    <joint name="ned_frame_joint" type="fixed">
-      <child link="ned_frame" />
-      <parent link="world" />
-      <origin xyz="0.0 0.0 0.0" rpy="${pi} 0 0"/>
-    </joint>
   </xacro:macro>
 </robot>

Commit message: set_max_param attempt

File: description/ros2_control/vehicle_system_multi_interface.ros2_control.xacro (robot description, xacro)
@@ -1,5 +1,5 @@
 <?xml version="1.0"?>
 <robot xmlns:xacro="http://www.ros.org/wiki/xacro">
-  <xacro:macro name="vehicle_system_multi_interface" params="name prefix serial_port state_update_frequency use_hardware frame_id child_frame_id map_frame_id">
+  <xacro:macro name="vehicle_system_multi_interface" params="name prefix serial_port state_update_frequency use_hardware frame_id child_frame_id map_frame_id max_set_param_attempts">
     <ros2_control name="${name}" type="system">
       <hardware>
@@ -10,4 +10,5 @@
           <param name="child_frame_id">${child_frame_id}</param>
           <param name="map_frame_id">${map_frame_id}</param>
+          <param name="max_set_param_attempts">${max_set_param_attempts}</param>
         </xacro:if>
         <xacro:unless value="${use_hardware}">

File: description/xacro/robot_system_multi_interface.urdf.xacro (robot description, xacro)
@@ -61,5 +61,6 @@
       frame_id="base_link"
       child_frame_id="${prefix}base_link"
-      map_frame_id="${prefix}map"/>
+      map_frame_id="${prefix}map"
+      max_set_param_attempts="5"/>
       <!-- Recursively call the macro for the next robot -->
       <xacro:instantiate_robots index="${index + 1}" count="${count}"/>
@@ -93,5 +94,6 @@
       frame_id="base_link"
       child_frame_id="${prefix}base_link"
-      map_frame_id="${prefix}map"/>
+      map_frame_id="${prefix}map"
+      max_set_param_attempts="5"/>
   </xacro:if>
 </robot>

Commit message: removed kf node and implement internal fusion

File: description/ros2_control/vehicle_system_multi_interface.ros2_control.xacro (robot description, xacro)
@@ -191,14 +191,24 @@
         <state_interface name="sim_time"/>
         <state_interface name="sim_period"/>
-        <state_interface name="imu_position_x"/>
-        <state_interface name="imu_position_y"/>
-        <state_interface name="imu_position_z"/>
+        <state_interface name="imu_roll"/>
+        <state_interface name="imu_pitch"/>
+        <state_interface name="imu_yaw"/>
         <state_interface name="imu_orientation_w"/>
         <state_interface name="imu_orientation_x"/>
         <state_interface name="imu_orientation_y"/>
         <state_interface name="imu_orientation_z"/>
+        <state_interface name="imu_angular_vel_x"/>
+        <state_interface name="imu_angular_vel_y"/>
+        <state_interface name="imu_angular_vel_z"/>
+        <state_interface name="imu_linear_acceleration_x"/>
+        <state_interface name="imu_linear_acceleration_y"/>
+        <state_interface name="imu_linear_acceleration_z"/>
+        <state_interface name="depth_from_pressure2"/>
         <state_interface name="dvl_gyro_roll"/>
         <state_interface name="dvl_gyro_pitch"/>
         <state_interface name="dvl_gyro_yaw"/>
+        <state_interface name="dvl_speed_x"/>
+        <state_interface name="dvl_speed_y"/>
+        <state_interface name="dvl_speed_z"/>
       </gpio>
     </ros2_control>

File: description/xacro/urdf.xacro (robot description, xacro)
@@ -63,5 +63,5 @@
     </joint>
     <joint name="${prefix}manipulator_mount_joint" type="fixed">
-      <origin rpy="0 0 0" xyz="0.14 0.0 -0.12" />
+      <origin rpy="0 0 0" xyz="0.19 0.0 -0.12" />
       <parent link="${prefix}base_link" />
       <child link="${prefix}manipulator_mount_link" />
